File: pcb/ATMEGA328_Motor_Board.kicad_pcb (KiCad board)
At the start: 2 copper layers, 77 x 100 mm, 259 parts, among them P1 CONN_01X04, P10 CONN_01X04, P11 CONN_01X02, P12 CONN_01X03, P13 CONN_01X02, P14 USB_MINI, P15 CONN_01X03, P16 CONN_02X03, P2 CONN_01X04, P3 CONN_01X03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

Commit message: Update to Kicad 7.0
Other:
- net class Default removed
- net class Potencia removed
